Commit message: update for fellowme and fix description

File: fellowme_description/urdf/fellowme_description.urdf (robot description, URDF)
Before this commit: robot fellowme_description, 4 links, 3 joints
Links:
- link base_link: mass 1.8441 -> 1.84414105853374
- link wheel_right: mass 1.8441 -> 0.12826
Joints:
- joint wheel_left_joint: origin xyz=0 0.13932 -0.075148 rpy=-1.6144 0 0 -> xyz=0 0.14246 -0.069 rpy=-1.5708 0 0
- joint wheel_right_joint: origin xyz=0 -0.15633 -0.06224 rpy=1.5272 0 0 -> xyz=0 -0.15346 -0.069 rpy=1.5708 0 0
